File: pcb/FeederController.kicad_pcb (KiCad board)
At the start: 4 copper layers, 100 x 100 mm, 103 parts, among them J1 Feeder 1, J10 Feeder 10, J11 Feeder 11, J12 Feeder 12, J13 Feeder 13, J14 Feeder 14, J15 Feeder 15, J16 Feeder 16, J17 12-24v DC, J18 5V Supply, J19 Feeder 17, J2 Feeder 2, J20 Feeder 18, J21 Feeder 19, J22 Feeder 20, J23 Feeder 21, J24 Feeder 22, J25 Feeder 23, J26 Feeder 24, J27 Feeder 25, J28 Feeder 26, J29 Feeder 27, J3 Feeder 3, J30 Feeder 28, J31 Feeder 29, J32 Feeder 30, J33 Feeder 31, J34 Feeder 32, J35 EXT-I2C, J4 Feeder 4, J5 Feeder 5, J6 Feeder 6, J7 Feeder 7, J8 Feeder 8, J9 Feeder 9, Q1 DMP3028LK3-13, U1 ESP32-Module, U2 PCA9685PW, U3 MCP23017, U4 AP2114-3.3, U5 AP63205WU, U6 PCA9685PW, U7 MCP23017_ML

Commit message: Changes to be committed: 	modified:   ../pcb/FeederController.kicad_pcb 	modified:   ../pcb/FeederController.kicad_prl 	modified:   ../pcb/FeederController.kicad_pro 	modified:   ../pcb/FeederController.kicad_sch 	deleted:    ../pcb/Outputs/Esp32FeederController-v1.0.0.zip 	modified:   ../pcb/fp-info-cache 	modified:   ../pcb/power.kicad_sch 	modified:   ../pcb/servo1.kicad_sch 	modified:   ../pcb/servo2.kicad_sch
 Untracked files:
	../pcb/FeederController.csv
	../pcb/FeederController.xml
Parts:
- removed R18, R3, R9: 10K, Resistor_SMD:R_0603_1608Metric_Pad0.98x0.95mm_HandSolder
- added J19: Feeder 17, Connector_PinHeader_2.54mm:PinHeader_1x04_P2.54mm_Vertical, F.Cu at (109.2, 84.5)
- added J35: Feeder 17, Connector_PinHeader_2.54mm:PinHeader_1x04_P2.54mm_Vertical, F.Cu at (109.2, 97.3)
- added LED1: PinHeader_1x03_P2.54mm_Vertical, Connector_PinHeader_2.54mm:PinHeader_1x03_P2.54mm_Vertical, F.Cu at (142.3, 47.5)
- added LED1: PinHeader_1x03_P2.54mm_Vertical, Connector_PinHeader_2.54mm:PinHeader_1x03_P2.54mm_Vertical, F.Cu at (162.6, 137.2)
- added LED2: PinHeader_1x03_P2.54mm_Vertical, Connector_PinHeader_2.54mm:PinHeader_1x03_P2.54mm_Vertical, F.Cu at (175.3, 137.2)
- added REF**: SolderJumper-2_P1.3mm_Open_Pad1.0x1.5mm, Jumper:SolderJumper-2_P1.3mm_Open_Pad1.0x1.5mm, F.Cu at (114.0, 105.0)
- moved REF** 1.78 mm to (171.4, 125.3)
- renumbered J35 to J36
Connections:
- U2 pad 23: Net-(U2-Pad23) -> GND
- U2 pad 24: unconnected-(U2-Pad24) -> GND
- U2 pad 3: unconnected-(U2-Pad3) -> GND
- U2 pad 4: unconnected-(U2-Pad4) -> GND
- U2 pad 5: unconnected-(U2-Pad5) -> GND
- U3 pad 11: Net-(U3-Pad11) -> GND
- U3 pad 13: unconnected-(U3-Pad13) -> GND
- U6 pad 23: Net-(R9-Pad2) -> GND
- U6 pad 24: unconnected-(U6-Pad24) -> GND
- U6 pad 4: unconnected-(U6-Pad4) -> GND
- U6 pad 5: unconnected-(U6-Pad5) -> GND
- U7 pad 13: unconnected-(U7-Pad13) -> GND
Routing:
- net unconnected-(U1-Pad27): track 0.00 -> 109.0 mm, vias 0 -> 2
- net unconnected-(U1-Pad13): track 0.00 -> 88.0 mm, vias 0 -> 2
- net +5V: track 265.4 -> 326.6 mm
- net unconnected-(U1-Pad5V): track 41.9 -> 3.61 mm
- net GND: track 34.9 -> 72.7 mm, vias 73 -> 76
- net unconnected-(U1-Pad19): track 2.60 -> 34.9 mm
- net unconnected-(U1-Pad25): track 0.00 -> 20.9 mm
- net unconnected-(U1-Pad26): track 0.00 -> 20.7 mm
- net unconnected-(U1-Pad32): track 0.00 -> 18.0 mm
- net unconnected-(U1-Pad33): track 0.00 -> 12.6 mm
- net +3V3: track 277.9 -> 285.9 mm
- net (no net): track 0.00 -> 7.80 mm
- net Net-(U3-Pad11): track 3.56 -> 0.00 mm
- net Net-(U2-Pad23): track 2.00 -> 0.00 mm
- net Net-(R9-Pad2): track 1.96 -> 0.00 mm
Other:
- board text added: "13"
- board text added: "19"
- board text added: "27"
- board text added: "5V"
- board text added: "J37"
- board text removed: "JLCJLCJLCJLC"
- board text removed: "Mounting holes are centered at 90mm apart in all directions. This allows easy mounting to the LumenPnP staging plate."
- board text removed: "https://atanisoft.github.com/Esp32FeederController"
