File: pcb/FeederController.kicad_sch (KiCad schematic)
At the start: 13 parts, among them J35 EXT-I2C, U1 ESP32-Module

Commit message: Changes to be committed: 	modified:   ../pcb/FeederController.kicad_pcb 	modified:   ../pcb/FeederController.kicad_prl 	modified:   ../pcb/FeederController.kicad_pro 	modified:   ../pcb/FeederController.kicad_sch 	deleted:    ../pcb/Outputs/Esp32FeederController-v1.0.0.zip 	modified:   ../pcb/fp-info-cache 	modified:   ../pcb/power.kicad_sch 	modified:   ../pcb/servo1.kicad_sch 	modified:   ../pcb/servo2.kicad_sch
 Untracked files:
	../pcb/FeederController.csv
	../pcb/FeederController.xml
Connections:
- no-connect marks 26 -> 24
