File: pcb/servo1.kicad_sch (KiCad schematic)
At the start: 34 parts, among them J1 Feeder 1, J10 Feeder 10, J11 Feeder 11, J12 Feeder 12, J13 Feeder 13, J14 Feeder 14, J15 Feeder 15, J16 Feeder 16, J2 Feeder 2, J3 Feeder 3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

Commit message: Changes to be committed: 	modified:   ../pcb/FeederController.kicad_pcb 	modified:   ../pcb/FeederController.kicad_prl 	modified:   ../pcb/FeederController.kicad_pro 	modified:   ../pcb/FeederController.kicad_sch 	deleted:    ../pcb/Outputs/Esp32FeederController-v1.0.0.zip 	modified:   ../pcb/fp-info-cache 	modified:   ../pcb/power.kicad_sch 	modified:   ../pcb/servo1.kicad_sch 	modified:   ../pcb/servo2.kicad_sch
 Untracked files:
	../pcb/FeederController.csv
	../pcb/FeederController.xml
Parts:
- removed R18: 10K, Resistor_SMD:R_0603_1608Metric_Pad0.98x0.95mm_HandSolder, symbol Device:R_Small_US
Connections:
- net GND: now also U2.24 (A5), U2.3 (A2), U2.4 (A3), U2.5 (A4), U3.11 (A0), U3.13 (A2)
- no-connect marks 5 -> 0
