File: pcb/servo2.kicad_sch (KiCad schematic)
At the start: 35 parts, among them J19 Feeder 17, J20 Feeder 18, J21 Feeder 19, J22 Feeder 20, J23 Feeder 21, J24 Feeder 22, J25 Feeder 23, J26 Feeder 24, J27 Feeder 25, J28 Feeder 26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

Commit message: Changes to be committed: 	modified:   ../pcb/FeederController.kicad_pcb 	modified:   ../pcb/FeederController.kicad_prl 	modified:   ../pcb/FeederController.kicad_pro 	modified:   ../pcb/FeederController.kicad_sch 	deleted:    ../pcb/Outputs/Esp32FeederController-v1.0.0.zip 	modified:   ../pcb/fp-info-cache 	modified:   ../pcb/power.kicad_sch 	modified:   ../pcb/servo1.kicad_sch 	modified:   ../pcb/servo2.kicad_sch
 Untracked files:
	../pcb/FeederController.csv
	../pcb/FeederController.xml
Connections:
- net GND: now also U6.24 (A5), U6.4 (A3), U6.5 (A4), U7.13 (A2)
- no-connect marks 4 -> 0
